Commit message: Added new example and new world file...stil working on it

File: tests/robots/coman/coman.urdf (robot description, URDF)
Before this commit: robot coman, 64 links, 63 joints
Joints:
- joint imu_joint: origin xyz=-0.072 -0.0068 0.044 rpy=0 3.14159265359 0 -> xyz=-0.072 -0.0068 0.044 rpy=0 0 0
