Commit message: ported panda ik

File: tests/robots/panda/panda.urdf (robot description, URDF)
Before this commit: robot panda, 10 links, 9 joints
Links:
- removed link panda_link0
- removed link panda_link1
- removed link panda_link2
- removed link panda_link3
- removed link panda_link4
- removed link panda_link5
- removed link panda_link6
- removed link panda_link7
- removed link panda_link8
- added link fp3_link0; collision cylinder length=0.03 radius=0.09; collision sphere radius=0.09
- added link fp3_link1; collision cylinder length=0.2830 radius=0.09; collision sphere radius=0.09
- added link fp3_link2; collision cylinder length=0.12 radius=0.09; collision sphere radius=0.09
- added link fp3_link3; collision cylinder length=0.15 radius=0.09; collision sphere radius=0.09
- added link fp3_link4; collision cylinder length=0.12 radius=0.09; collision sphere radius=0.09
- added link fp3_link5; collision cylinder length=0.1 radius=0.09; collision cylinder length=0.14 radius=0.055
- added link fp3_link6; collision cylinder length=0.08 radius=0.08; collision sphere radius=0.08
- added link fp3_link7; collision cylinder length=0.14 radius=0.07; collision sphere radius=0.07
- added link fp3_link8; collision cylinder length=0.01 radius=0.06; collision sphere radius=0.06
Joints:
- removed joint panda_joint1
- removed joint panda_joint2
- removed joint panda_joint3
- removed joint panda_joint4
- removed joint panda_joint5
- removed joint panda_joint6
- removed joint panda_joint7
- removed joint panda_joint8
- added joint fp3_joint1: type revolute, parent fp3_link0, child fp3_link1, origin xyz=0 0 0.333 rpy=0 0 0, axis 0 0 1, limit lower=-2.8973 upper=2.8973 effort=87 velocity=2.1750
- added joint fp3_joint2: type revolute, parent fp3_link1, child fp3_link2, origin xyz=0 0 0 rpy=-1.5707963267948966 0 0, axis 0 0 1, limit lower=-1.7628 upper=1.7628 effort=87 velocity=2.1750
- added joint fp3_joint3: type revolute, parent fp3_link2, child fp3_link3, origin xyz=0 -0.316 0 rpy=1.5707963267948966 0 0, axis 0 0 1, limit lower=-2.8973 upper=2.8973 effort=87 velocity=2.1750
- added joint fp3_joint4: type revolute, parent fp3_link3, child fp3_link4, origin xyz=0.0825 0 0 rpy=1.5707963267948966 0 0, axis 0 0 1, limit lower=-3.0718 upper=-0.0698 effort=87 velocity=2.1750
- added joint fp3_joint5: type revolute, parent fp3_link4, child fp3_link5, origin xyz=-0.0825 0.384 0 rpy=-1.5707963267948966 0 0, axis 0 0 1, limit lower=-2.8973 upper=2.8973 effort=12 velocity=2.6100
- added joint fp3_joint6: type revolute, parent fp3_link5, child fp3_link6, origin xyz=0 0 0 rpy=1.5707963267948966 0 0, axis 0 0 1, limit lower=-0.0175 upper=3.7525 effort=12 velocity=2.6100
- added joint fp3_joint7: type revolute, parent fp3_link6, child fp3_link7, origin xyz=0.088 0 0 rpy=1.5707963267948966 0 0, axis 0 0 1, limit lower=-2.8973 upper=2.8973 effort=12 velocity=2.6100
- added joint fp3_joint8: type fixed, parent fp3_link7, child fp3_link8, origin xyz=0 0 0.107 rpy=0 0 0
- joint world_joint: child panda_link0 -> fp3_link0
